File: Core.kicad_sch (KiCad schematic)
At the start: 34 parts, among them J14 Solder Jumper, U1 AUDIO_CLK_GEN, U2 TPS63001DRCR, U3 STM32U575RGT6

Commit message: power planes
Parts:
- removed 3V3, GND1: Test Pad, TestPoint:TestPoint_Pad_D1.0mm, symbol gap9_deck:root_0_CMP-01283-1_gap9_deck.SCHLIB
- removed BVBAT1: Test Pad, TestPoint:TestPoint_Pad_D1.0mm, symbol gap9_deck:root_3_CMP-01283-1_gap9_deck.SCHLIB
- added 3V3: 3V3, Connector_PinHeader_2.54mm:PinHeader_1x01_P2.54mm_Vertical, symbol Connector:Conn_01x01_Socket
- added GND1, VBAT1: GND1, Connector_PinHeader_2.54mm:PinHeader_1x01_P2.54mm_Vertical, symbol Connector:Conn_01x01_Socket
- added J21: Solder Jumper, Jumper:SolderJumper-2_P1.3mm_Open_RoundedPad1.0x1.5mm, symbol gap9_deck:CMP-00005-5
Connections:
- net 3V3: now also 3V3.1 (Pin_1), J21.1; no longer C1.1, C10.2, C11.1, C13.2, C16.1, C3.1, C6.1, C8.2, C9.2, R5.1, R6.1, U1.1 (INH), U1.4 (VCC), U3.1 (VBAT), U3.13 (VDDA), U3.19 (VDD), U3.32 (VDD), U3.48 (VDDUSB), U3.64 (VDD)
- net GND: now also GND1.1 (Pin_1)
- net VBat: now also VBAT1.1 (Pin_1)
- new net VCORE: C1.1, C10.2, C11.1, C13.2, C16.1, C3.1, C6.1, C8.2, C9.2, J21.2, R5.1, R6.1, U1.1 (INH), U1.4 (VCC), U3.1 (VBAT), U3.13 (VDDA), U3.19 (VDD), U3.32 (VDD), U3.48 (VDDUSB), U3.64 (VDD)
Other:
- moved on the sheet: J14
