File: microphones.kicad_sch (KiCad schematic)
At the start: 31 parts, among them J10 Molex expansions, J11 Molex expansions, J12 Molex expansions, J13 Molex expansions, J15 Solder Jumper, J16 Solder Jumper, J17 Solder Jumper, J2 Solder Jumper, J3 Solder Jumper, J4 Solder Jumper, J5 Solder Jumper, J6 Solder Jumper, J7 Solder Jumper, J8 Solder Jumper, J9 Solder Jumper, M1 Microphone, M2 Microphone, M3 Microphone, M4 Microphone, M5 Microphone, M7 Microphone

Commit message: power planes
Parts:
- added J19: Solder Jumper, Jumper:SolderJumper-2_P1.3mm_Open_RoundedPad1.0x1.5mm, symbol gap9_deck:CMP-00005-5
Connections:
- net 3V3: now also J19.1; no longer C23.1, C24.1, C25.1, C26.1, C27.1, C29.1, J10.1, J11.1, J12.1, J13.1, M1.1 (VDD), M2.1 (VDD), M3.1 (VDD), M3.4 (L/R), M4.1 (VDD), M4.4 (L/R), M5.1 (VDD), M7.1 (VDD), M7.4 (L/R)
- new net VMIC: C23.1, C24.1, C25.1, C26.1, C27.1, C29.1, J10.1, J11.1, J12.1, J13.1, J19.2, M1.1 (VDD), M2.1 (VDD), M3.1 (VDD), M3.4 (L/R), M4.1 (VDD), M4.4 (L/R), M5.1 (VDD), M7.1 (VDD), M7.4 (L/R)
