File: connectors.kicad_sch (KiCad schematic)
At the start: 45 parts, among them J1 Micro-SD Slot, P1 Crazyflie Female Expansion, P2 Crazyflie Female Expansion, P3 6220XX21121_62201021121, SW1 Test Pad, U4 DS28E05R+T

Commit message: power planes
Parts:
- added J20: Solder Jumper, Jumper:SolderJumper-2_P1.3mm_Open_RoundedPad1.0x1.5mm, symbol gap9_deck:CMP-00005-5
Connections:
- net 3V3: now also J20.1; no longer C20.1, C21.2, J1.4 (VDD), P3.1, R14.2, R15.2, R16.2, R17.2, R18.2, R19.1, R22.2
- new net VCORE: P3.1, R22.2
- new net VSD: C20.1, C21.2, J1.4 (VDD), J20.2, R14.2, R15.2, R16.2, R17.2, R18.2, R19.1
